Commit message: Simple joint space planning for IRB360-800

File: abb_irb360_support/urdf/abb_irb360_support.urdf (robot description, URDF)
Before this commit: robot abb_irb360_support, 7 links, 6 joints
Links:
- added link upper_arm_2, mass 0; collision mesh filename=package://abb_irb360_support/meshes/upper_arm_2.STL; visual mesh filename=package://abb_irb360_support/meshes/upper_arm_2.STL
- added link upper_arm_3, mass 0; collision mesh filename=package://abb_irb360_support/meshes/upper_arm_3.STL; visual mesh filename=package://abb_irb360_support/meshes/upper_arm_3.STL
- added link upper_universal_link_2, mass 0; collision mesh filename=package://abb_irb360_support/meshes/upper_universal_link_2.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; visual mesh filename=package://abb_irb360_support/meshes/upper_universal_link_2.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
- added link upper_universal_link_3, mass 0; collision mesh filename=package://abb_irb360_support/meshes/upper_universal_link_3.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; visual mesh filename=package://abb_irb360_support/meshes/upper_universal_link_3.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
- link base_link: mass None -> 49.2535162198679
- link end_link: mass None -> 0.020194
- link lower_arm_1: mass None -> 0.13022
- link lower_universal_link_1: mass None -> 0.0087708
- link moving_platform: mass None -> 0.12295
- link upper_arm_1: mass None -> 0.91849
- link upper_universal_link_1: mass None -> 0.0087708
Joints:
- added joint joint_2: type fixed, parent base_link, child upper_arm_2, origin xyz=-0.1 -0.17321 -0.275 rpy=0 -0.11527 -2.0944, axis 0 0 0
- added joint joint_3: type fixed, parent base_link, child upper_arm_3, origin xyz=-0.1 0.17321 -0.275 rpy=0 -0.11527 2.0944, axis 0 0 0
- added joint uj_21: type fixed, parent upper_arm_2, child upper_universal_link_2, origin xyz=0.23344 0 -0.027 rpy=-1.5708 0.9463 3.1416, axis 0 0 0
- added joint uj_31: type fixed, parent upper_arm_3, child upper_universal_link_3, origin xyz=0.23344 0 -0.027 rpy=-1.5708 0.9463 -3.1416, axis 0 0 0
- joint joint_1: origin xyz=0.2 0 -0.275 rpy=0 -0.11527 0 -> xyz=0.2 0 -0.275 rpy=0 -0.115268716889166 0
- joint joint_4: origin xyz=-0.045 0 0 rpy=0 0 0 -> xyz=-0.0449999999999976 0 0 rpy=0 0 0
- joint uj_11: origin xyz=0.23344 0 -0.027 rpy=0 0.62449 0 -> xyz=0.233443783382638 0 -0.0269999999999995 rpy=0 0.624492885969242 0
- joint uj_12: origin xyz=0 0 0 rpy=1.5708 1.5708 0 -> xyz=0 0 0 rpy=1.5707963267949 1.5707963267949 0
- joint uj_13: origin xyz=0.8 0 0 rpy=-1.5708 0 -1.5708 -> xyz=0.799999999999999 0 0 rpy=-1.5707963267949 0 -1.5707963267949
- joint uj_14: origin xyz=0 0 0 rpy=-3.1416 0.50922 -3.1416 -> xyz=0 0 0 rpy=-3.14159265358979 0.509224169080082 -3.14159265358979

File: abb_irb360_support/urdf/irb360_800.urdf.xacro (robot description, xacro)
@@ -2,4 +2,16 @@
 <robot xmlns:xacro="http://ros.org/wiki/xacro" name="irb360_800">
   <xacro:include filename="$(find abb_irb360_support)/urdf/irb360_800.xacro"/>
+  <xacro:include filename="$(find abb_irb360_support)/urdf/irb360_800_moving_platform.xacro"/>
+  <!-- Three arms macro -->
   <xacro:irb360_800 />
+  <!-- Attach moving platform to arm 1 -->
+  <xacro:irb360_800_moving_platform parent = "arm_1" theta = "1">
+    <origin xyz="0 0 0" rpy="-3.14159265358979 0.509224169080082 -3.14159265358979" />
+  </xacro:irb360_800_moving_platform>
+  <xacro:irb360_800_moving_platform parent = "arm_2" theta = "2">
+    <origin xyz="0 0 0" rpy="-3.14159265358979 0.509224169080082 -3.14159265358979" />
+  </xacro:irb360_800_moving_platform>
+  <xacro:irb360_800_moving_platform parent = "arm_3" theta = "3">
+    <origin xyz="0 0 0" rpy="-3.14159265358979 0.509224169080082 -3.14159265358979" />
+  </xacro:irb360_800_moving_platform>
 </robot>

File: abb_irb360_support/urdf/irb360_800.xacro (robot description, xacro)
@@ -3,4 +3,5 @@
   <xacro:include filename="$(find abb_irb360_support)/urdf/irb360_800_arm.xacro"/>
   <xacro:macro name="irb360_800">
+  <!-- Define base link -->
     <link name="base_link">
       <visual>
@@ -20,4 +21,5 @@
       </collision>
     </link>
+  <!-- Attach all arms to base link -->
     <xacro:irb360_800_arm arm="arm_1" theta="1">
       <origin xyz="0.2 0 -0.275" rpy="0 -0.11527 0" />
